File: i960SxSimpleBreakoutBoard.kicad_pcb (KiCad board)
At the start: 4 copper layers, 98.6 x 85.3 mm, 27 parts, among them J1 Conn_01x23, J2 Conn_02x16_Counter_Clockwise, J3 Data Lines, U1 74HC573, U2 74HC573, U3 80960Sx, U4 74HC245, U5 74HC245

Commit message: Finish the initial rev 2 design
Parts:
- moved D1 46.7 mm to (-46.6, -15.1), turned to 270 degrees
- moved R1 37.7 mm to (-47.7, -7.68), turned to 90 degrees
Routing:
- net /ALE: track 0.00 -> 115.5 mm, vias 0 -> 3
- net GND: track 164.1 -> 274.1 mm, vias 16 -> 19
- net /A31: track 0.00 -> 107.1 mm
- net /A30: track 0.00 -> 97.5 mm
- net /A29: track 0.00 -> 96.1 mm
- net /AD15: track 0.00 -> 93.6 mm, vias 0 -> 1
- net /A27: track 0.00 -> 93.0 mm
- net /A28: track 0.00 -> 92.6 mm
- net /A26: track 0.00 -> 90.6 mm
- net /~DEN: track 0.00 -> 89.6 mm, vias 0 -> 2
- net /A25: track 0.00 -> 87.7 mm
- net /AD14: track 0.00 -> 85.1 mm, vias 0 -> 1
- net /DT\~R: track 0.00 -> 84.3 mm, vias 0 -> 2
- net /A24: track 0.00 -> 82.9 mm
- net /A23: track 0.00 -> 80.0 mm
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- added copper zone on In1.Cu, net +5V
- added copper zone on In2.Cu, net GND
